File: sinope.sch (KiCad schematic (older format))
At the start: 33 parts, among them J1 PIOA, J2 PIOB, J3 SERIAL0, J4 SERIAL1, J5 Conn_01x02, U1 74LS04, U10 MAX232, U11 MAX232, U2 Z80CPU, U3 74LS32, U4 74LS138, U5 27128, U6 Z80CTC, U7 TC551001, U8 Z80SIO, U9 Z80PIO, Y1 3.6864

Commit message: SRAM Battery Backup
Parts:
- removed C1: 1uF, Capacitor_SMD:C_0805_2012Metric, symbol Device:C
- removed R1: 220K, Resistor_SMD:R_0805_2012Metric, symbol Device:R
- added C1: 100nF, symbol Device:C_Small
- added J6: Battery, symbol Connector_Generic:Conn_01x02
- added Q1: 2N3904, Package_TO_SOT_THT:TO-92_Inline, symbol Transistor_BJT:2N3904
- added R2: 3k3, symbol Device:R
- added unit 2 of U1
- added U7: MAX695, Package_DIP:DIP-16_W7.62mm, symbol sinope:MAX695
- J1: renamed from J5; value Conn_01x02 -> 5VDC
- renumbered J1 to J2, J2 to J3, J3 to J4, J4 to J5, R2 to R3, R3 to R4, U9 to U10, U8 to U11, U10 to U12, U11 to U13, U4 to U6, U6 to U8, U7 to U9
Connections:
- wire segments 340 -> 355
- no-connect marks 34 -> 41
Other:
- moved on the sheet: C10, C11, C12, C13, C4, C5, C6, C7, C8, C9, J1, J2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

Commit message: Video interface
Parts:
- added C14, C17, C18, C19, C20, C21: 100nF, symbol Device:C_Small
- added C15, C16: 16pF, symbol Device:C_Small
- added U14: TMS9929A, symbol sinope:TMS9929A
- added U15, U16, U18: 74HCT574, symbol 74xx:74HCT574
- added U17: HM62256BLP-7, DIP28, symbol sinope:HM62256BLP-7
- added U19: 74HCT04, symbol 74xx:74HCT04
- added U4: 74LS32, Package_DIP:DIP-14_W7.62mm, symbol 74xx:74LS32
- added Y2: 10.738635MHz, Crystal:Crystal_HC49-U_Horizontal, symbol Device:Crystal
Connections:
- net labels added: AD0, AD1, AD2, AD3, AD4, AD5, AD6, AD7, RD0, RD1, RD2, RD3, RD4, RD5, RD6, RD7, VA0, VA1, VA10, VA11, VA12, VA13, VA14, VA2, VA3, VA4, VA5, VA6, VA7, VA8, VA9, VIDEO_ADDRESS, VIDEO_DATA, ~NMI, ~VIDEOCS, ~WR
- wire segments 355 -> 548
Other:
- moved on the sheet: C10, C11, C12, C13, C4, C5, C6, C7, C8, C9, J4, J5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

Commit message: Rip out graphics
Parts:
- removed C16: 16pF, symbol Device:C_Small
- removed C17, C18, C19, C20, C21: 100nF, symbol Device:C_Small
- removed unit 2 of U1
- removed U14: TMS9929A, symbol sinope:TMS9929A
- removed U15, U16, U18: 74HCT574, symbol 74xx:74HCT574
- removed U17: HM62256BLP-7, DIP28, symbol sinope:HM62256BLP-7
- removed U19: 74HCT04, symbol 74xx:74HCT04
- removed U3, U4: 74LS32, Package_DIP:DIP-14_W7.62mm, symbol 74xx:74LS32
- removed U6: 74LS138, Package_DIP:DIP-16_W7.62mm, symbol 74xx:74LS138
- removed Y2: 10.738635MHz, Crystal:Crystal_HC49-U_Horizontal, symbol Device:Crystal
- added U3: SINOPE_GAL, symbol sinope:SINOPE_GAL
- C15: value 16pF -> 100nF
Connections:
- net labels added: CTSA, RAMVCC, RTSA, RxDA, TxDA, ~CTCCS, ~INT, ~MREQ, ~PIOCS, ~RAMCS, ~RAMCS_SAFE, ~ROMCS, ~SIOCS
- net labels removed: AD0, AD1, AD2, AD3, AD4, AD5, AD6, AD7, ADDRESS, DATA, RD0, RD1, RD2, RD3, RD4, RD5, RD6, RD7, VA0, VA1, VA10, VA11, VA12, VA13, VA14, VA2, VA3, VA4, VA5, VA6, VA7, VA8, VA9, VIDEO_ADDRESS, VIDEO_DATA, ~NMI, ~VIDEOCS
- wire segments 548 -> 345
- no-connect marks 41 -> 36
Other:
- moved on the sheet: C1, C10, C11, C12, C13, C4, C5, C6, C7, C8, C9, J1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

Commit message: Use integrated oscillator
Parts:
- removed C2, C3: 47pF, Capacitor_SMD:C_0805_2012Metric, symbol Device:C
- removed R3: 10M, Resistor_SMD:R_0805_2012Metric, symbol Device:R
- removed R4: 1k, Resistor_SMD:R_0805_2012Metric, symbol Device:R
- removed U1: 74LS04, Package_DIP:DIP-14_W7.62mm, symbol 74xx:74LS04
- removed Y1: 3.6864, Crystal:Crystal_HC49-U_Horizontal, symbol Device:Crystal
- added X1: 3.6864Mhz, Oscillator:Oscillator_DIP-14, symbol Oscillator:TFT680
Connections:
- wire segments 345 -> 337
Changed lines of the file:
@@
 Text GLabel 2900 7150 2    50   Output ~ 0
 ~RESET
-$Comp
-L Device:C C2
-U 1 1 5EAE2B1A
-P 2250 1500
-F 0 "C2" H 2365 1546 50  0000 L CNN
-F 1 "47pF" H 2365 1455 50  0000 L CNN
-F 2 "Capacitor_SMD:C_0805_2012Metric" H 2288 1350 50  0001 C CNN
-F 3 "~" H 2250 1500 50  0001 C CNN
-	1    2250 1500
-	1    0    0    -1
-$EndComp
-$Comp
-L Device:C C3
-U 1 1 5EAE32B1
-P 2800 1500
-F 0 "C3" H 2915 1546 50  0000 L CNN
-F 1 "47pF" H 2915 1455 50  0000 L CNN
-F 2 "Capacitor_SMD:C_0805_2012Metric" H 2838 1350 50  0001 C CNN
-F 3 "~" H 2800 1500 50  0001 C CNN
-	1    2800 1500
-	1    0    0    -1
-$EndComp
-$Comp
-L Device:R R3
-U 1 1 5EAE40DE
-P 2250 1000
-F 0 "R3" H 2050 1050 50  0000 L CNN
-F 1 "10M" H 2050 950 50  0000 L CNN
-F 2 "Resistor_SMD:R_0805_2012Metric" V 2180 1000 50  0001 C CNN
-F 3 "~" H 2250 1000 50  0001 C CNN
-	1    2250 1000
-	1    0    0    -1
-$EndComp
-$Comp
-L Device:R R4
-U 1 1 5EAE4756
-P 2800 1000
-F 0 "R4" H 2870 1046 50  0000 L CNN
-F 1 "1k" H 2870 955 50  0000 L CNN
-F 2 "Resistor_SMD:R_0805_2012Metric" V 2730 1000 50  0001 C CNN
-F 3 "~" H 2800 1000 50  0001 C CNN
-	1    2800 1000
-	1    0    0    -1
-$EndComp
-$Comp
-L Device:Crystal Y1
-U 1 1 5EAE53AE
-P 2550 1250
-F 0 "Y1" H 2550 1518 50  0000 C CNN
-F 1 "3.6864" H 2550 1427 50  0000 C CNN
-F 2 "Crystal:Crystal_HC49-U_Horizontal" H 2550 1250 50  0001 C CNN
-F 3 "~" H 2550 1250 50  0001 C CNN
-	1    2550 1250
-	1    0    0    -1
-$EndComp
-$Comp
-L 74xx:74LS04 U1
-U 1 1 5EAED368
-P 1850 1250
-F 0 "U1" H 1850 1550 50  0000 C CNN
-F 1 "74LS04" H 1850 1450 50  0000 C CNN
-F 2 "Package_DIP:DIP-14_W7.62mm" H 1850 1250 50  0001 C CNN
-F 3 "http://www.ti.com/lit/gpn/sn74LS04" H 1850 1250 50  0001 C CNN
-	1    1850 1250
-	-1   0    0    1
-$EndComp
-Wire Wire Line
-	1550 1250 1550 2600
 Wire Wire Line
 	1550 2600 1850 2600
-Wire Wire Line
-	2150 1250 2250 1250
-Wire Wire Line
-	2250 1250 2250 1150
-Connection ~ 2250 1250
-Wire Wire Line
-	2250 1250 2400 1250
-Wire Wire Line
-	2250 1350 2250 1250
-Wire Wire Line
-	2700 1250 2800 1250
-Wire Wire Line
-	2800 1250 2800 1150
-Wire Wire Line
-	2800 1250 2800 1350
-Connection ~ 2800 1250
-Wire Wire Line
-	2250 1650 2800 1650
-$Comp
-L power:GND #PWR09
-U 1 1 5EB1616A
-P 2800 1650
-F 0 "#PWR09" H 2800 1400 50  0001 C CNN
-F 1 "GND" H 2805 1477 50  0000 C CNN
-F 2 "" H 2800 1650 50  0001 C CNN
-F 3 "" H 2800 1650 50  0001 C CNN
-	1    2800 1650
-	1    0    0    -1
-$EndComp
-Wire Wire Line
-	1550 1250 1550 750
-Wire Wire Line
-	1550 750  2250 750
-Wire Wire Line
-	2250 750  2250 850
-Connection ~ 1550 1250
-Wire Wire Line
-	2250 750  2800 750
-Wire Wire Line
-	2800 750  2800 850
-Connection ~ 2250 750
-Connection ~ 2800 1650
 Text GLabel 1800 3300 0    50   Output ~ 0
 ~M1
-Text GLabel 1000 1250 0    50   Output ~ 0
+Text GLabel 1650 1250 2    50   Output ~ 0
 CLK
-Wire Wire Line
-	1000 1250 1550 1250
 Entry Wire Line
 	3750 2200 3650 2300
@@
 Wire Wire Line
 	4900 4200 4900 4250
+$Comp
+L power:GND #PWR03
+U 1 1 5F85FCD9
+P 1250 1600
+F 0 "#PWR03" H 1250 1350 50  0001 C CNN
+F 1 "GND" H 1255 1427 50  0000 C CNN
+F 2 "" H 1250 1600 50  0001 C CNN
+F 3 "" H 1250 1600 50  0001 C CNN
+	1    1250 1600
+	1    0    0    -1
+$EndComp
+$Comp
+L power:+5V #PWR02
+U 1 1 5F860570
+P 1250 900
+F 0 "#PWR02" H 1250 750 50  0001 C CNN
+F 1 "+5V" H 1265 1073 50  0000 C CNN
+F 2 "" H 1250 900 50  0001 C CNN
+F 3 "" H 1250 900 50  0001 C CNN
+	1    1250 900
+	1    0    0    -1
+$EndComp
+$Comp
+L Oscillator:TFT680 X1
+U 1 1 5F81E577
+P 1250 1250
+F 0 "X1" H 1550 1600 50  0000 L CNN
+F 1 "3.6864Mhz" H 1400 1500 50  0000 L CNN
+F 2 "Oscillator:Oscillator_DIP-14" H 1700 900 50  0001 C CNN
+F 3 "http://cdn-reichelt.de/documents/datenblatt/B400/OSZI.pdf" H 1150 1250 50  0001 C CNN
+	1    1250 1250
+	1    0    0    -1
+$EndComp
+Wire Wire Line
+	1250 900  1250 950
+Wire Wire Line
+	1250 900  900  900
+Wire Wire Line
+	900  900  900  1250
+Wire Wire Line
+	900  1250 950  1250
+Connection ~ 1250 900
+Wire Wire Line
+	1550 1250 1550 2600
+Wire Wire Line
+	1550 1250 1650 1250
+Connection ~ 1550 1250
+Wire Wire Line
+	1250 1600 1250 1550
 Wire Bus Line
 	3650 2300 3650 3950

Commit message: Touchup
Parts:
- removed Q1: 2N3904, Package_TO_SOT_THT:TO-92_Inline, symbol Transistor_BJT:2N3904
- added C16, C17, C18, C19, C2, C20, C3: 100nF, Capacitor_SMD:C_0805_2012Metric, symbol Device:C_Small
- added D1: LED, LED_SMD:LED_0805_2012Metric, symbol Device:LED
- added Q1: 3N3906, Package_TO_SOT_THT:TO-92, symbol Device:Q_PNP_EBC
- added R1: 330, Resistor_SMD:R_0805_2012Metric, symbol Device:R
- added SW1: RESET, Button_Switch_THT:Push_E-Switch_KS01Q01, symbol Switch:SW_Push
- C1, C14, C15: footprint (none) -> Capacitor_SMD:C_0805_2012Metric
- J1: footprint (none) -> Connector_PinHeader_2.54mm:PinHeader_1x02_P2.54mm_Vertical
- J6: footprint (none) -> Connector_PinHeader_2.54mm:PinHeader_2x01_P2.54mm_Vertical
- R2: footprint (none) -> Resistor_SMD:R_0805_2012Metric
- U3: footprint (none) -> Package_DIP:DIP-24_W7.62mm
Connections:
- net labels added: SIOCA, SIOCB
- wire segments 337 -> 368
Other:
- moved on the sheet: C1, C14, J1, J6, U5, U7, U9

Commit message: Memory management logic
Parts:
- removed U3: SINOPE_GAL, Package_DIP:DIP-24_W7.62mm, symbol sinope:SINOPE_GAL
- removed U5: 27128, Package_DIP:DIP-28_W15.24mm, symbol Memory_EPROM:27128
- added C20, C21: 100nF, Capacitor_SMD:C_0805_2012Metric, symbol Device:C_Small
- added U10: MEMORY_GAL, symbol sinope:MEMORY_GAL
- added U11: 74LS157, symbol sinope:74LS157
- added U7: IO_GAL, symbol sinope:IO_GAL
- added U9: 27C010, symbol Memory_EPROM:27C010
- renumbered C8 to C1, C18 to C10, C17 to C11, C7 to C12, C11 to C13, C2 to C14, C19 to C16, C1 to C17, C3 to C18, C14 to C19, C4 to C2, C20 to C22, C12 to C3, C5 to C4, C9 to C5, C10 to C6, C6 to C7, C13 to C8, C16 to C9, J2 to J1, J4 to J2, J5 to J4, J6 to J5, J1 to J6, R2 to R1, R1 to R2, U2 to U1, U9 to U12, U8 to U2, U10 to U3, U11 to U4, U12 to U5, U13 to U6, U7 to U8
Connections:
- net labels added: RAMA16, ROMA14, ROMA15, ROMA16, ~BANKCS
- wire segments 368 -> 410
- no-connect marks 36 -> 38
Other:
- moved on the sheet: C18, C19, U12

Commit message: Package assignments, PCB work
Parts:
- U10, U7: footprint (none) -> Package_DIP:DIP-24_W7.62mm
- U11: footprint (none) -> Package_DIP:DIP-16_W7.62mm
- U9: footprint (none) -> Package_DIP:DIP-32_W15.24mm
Connections:
- no-connect marks 38 -> 37
Changed lines of the file:
@@
 U 1 1 5F7E8ED7
 P 13750 2950
-F 0 "C6" V 13500 3000 50  0000 C CNN
+F 0 "C6" V 13850 3050 50  0000 C CNN
 F 1 "100nF" V 13600 3000 50  0000 C CNN
 F 2 "Capacitor_SMD:C_0805_2012Metric" H 13750 2950 50  0001 C CNN
@@
 U 1 1 5F76B641
 P 13750 2450
-F 0 "C5" V 14000 2450 50  0000 C CNN
+F 0 "C5" V 13650 2350 50  0000 C CNN
 F 1 "100nF" V 13900 2450 50  0000 C CNN
 F 2 "Capacitor_SMD:C_0805_2012Metric" H 13750 2450 50  0001 C CNN
@@
 F 0 "U11" H 11000 8250 50  0000 C CNN
 F 1 "74LS157" H 11100 8150 50  0000 C CNN
-F 2 "" H 11000 8250 50  0001 C CNN
+F 2 "Package_DIP:DIP-16_W7.62mm" H 11000 8250 50  0001 C CNN
 F 3 "http://www.ti.com/lit/gpn/sn74LS157" H 11000 8250 50  0001 C CNN
 	1    11000 8400
@@
 F 0 "U9" H 7000 7400 50  0000 C CNN
 F 1 "27C010" H 7000 7300 50  0000 C CNN
-F 2 "" H 6900 7750 50  0001 C CNN
+F 2 "Package_DIP:DIP-32_W15.24mm" H 6900 7750 50  0001 C CNN
 F 3 "http://ww1.microchip.com/downloads/en/DeviceDoc/doc0321.pdf" H 6900 7750 50  0001 C CNN
 	1    6900 7750
@@
 	3650 6250 6200 6250
 NoConn ~ 3700 8750
-NoConn ~ 9400 5050
 Wire Wire Line
 	10150 9400 10250 9500
@@
 F 0 "U10" H 9150 8700 50  0000 C CNN
 F 1 "MEMORY_GAL" H 9150 8600 50  0000 C CNN
-F 2 "" H 9050 8900 50  0001 C CNN
+F 2 "Package_DIP:DIP-24_W7.62mm" H 9050 8900 50  0001 C CNN
 F 3 "" H 9050 8900 50  0001 C CNN
 	1    9100 8900
@@
 F 0 "U7" H 4950 5000 50  0000 C CNN
 F 1 "IO_GAL" H 5000 4900 50  0000 C CNN
-F 2 "" H 4900 5100 50  0001 C CNN
+F 2 "Package_DIP:DIP-24_W7.62mm" H 4900 5100 50  0001 C CNN
 F 3 "" H 4900 5100 50  0001 C CNN
 	1    4900 5100
