File: CompositeModulator.sch (KiCad schematic (older format))
At the start: 51 parts, among them Q2 9015, Q3 9014, U13 TBA520, U14 74LS04, Y1 4.433618 Mhz

Commit message: Add composite modulator PCB as test project
Parts:
- added J1: Input, Connector_PinHeader_2.54mm:PinHeader_1x05_P2.54mm_Vertical, symbol Connector:Conn_01x05_Male
- added J2: Composite Video, Connector_PinHeader_2.54mm:PinHeader_1x02_P2.54mm_Vertical, symbol Connector:Conn_Coaxial
- C23, C24, C25, C26, C27, C28, C29, C30, C31, C32, C33, C34, C35, C36, C37, C38, C40, C41, C43, C44, C45: footprint (none) -> Capacitor_SMD:C_0805_2012Metric
- C39: footprint (none) -> Capacitor_SMD:C_Trimmer_Murata_TZC3
- L1, L2: footprint (none) -> Inductor_SMD:L_0805_2012Metric
- L3: footprint (none) -> Inductor_THT:L_Toroid_Vertical_L10.0mm_W5.0mm_P5.08mm
- Q2, Q3: footprint (none) -> Package_TO_SOT_THT:TO-92
- R10, R12, R13, R14, R15, R16, R18, R19, R20, R21, R22, R3, R4, R5, R6, R7, R8, R9: footprint (none) -> Resistor_SMD:R_0805_2012Metric
- R11, R17: footprint (none) -> Potentiometer_THT:Potentiometer_Piher_PT-6-V_Vertical
- U13: footprint (none) -> Package_DIP:DIP-16_W7.62mm
- U14: footprint (none) -> Package_DIP:DIP-14_W7.62mm
- Y1: footprint (none) -> Crystal:Crystal_HC49-U_Vertical
- renumbered C42 to C1
Connections:
- net labels removed: CVID
- wire segments 153 -> 164
Other:
- moved on the sheet: C1, C23, C24, C25, C26, C27, C28, C29, C30, C31, C32, C33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
