File: hardware/sinope.kicad_pcb (KiCad board)
At the start: 2 copper layers, 160 x 100 mm, 52 parts, among them J1 PIOA, J2 SERIAL1, J3 PIOB, J4 USB_B_Micro, J7 Z80_BUS, Q1 MMBT3904, SW1 RESET, U1 Z80CPU, U10 MEMORY_GAL, U11 74LS157, U12 TC551001, U2 Z80CTC, U3 Z80PIO, U4 Z80SIO, U5 MAX232, U6 FT232RL, U7 IO_GAL, U8 MAX695, U9 27C010, X1 3.6864Mhz

Commit message: Layout redone quickly
Parts:
- moved C19 119.8 mm to (80.5, 53.6), turned to 0 degrees
- moved C6 112.3 mm to (193.2, 79.1)
- moved C11 92.4 mm to (123.8, 95.2)
- moved J4 74.8 mm to (42.0, 34.0)
- moved C16 69.1 mm to (166.4, 79.8), turned to 180 degrees
- moved C10 65.5 mm to (149.9, 103.8)
- moved C18 64.6 mm to (164.6, 38.1), turned to 0 degrees
- moved C17 60.3 mm to (63.8, 30.4)
- moved SW1 59.8 mm to (45.0, 111.9)
- moved X1 57.9 mm to (101.3, 36.6)
- moved C5 56.2 mm to (136.9, 93.8)
- moved C14 54.4 mm to (75.9, 45.1)
- moved C20 51.8 mm to (93.5, 100.1), turned to 180 degrees
- moved C15 46.8 mm to (80.7, 60.1), turned to 0 degrees
- moved J2 44.1 mm to (42.7, 43.6)
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Connections:
- JP1 pad 2: /ROMA16 -> Net-(JP1-Pad2)
- JP2 pad 2: ~RD -> Net-(JP2-Pad2)
- U9 pad 2: /ROMA16 -> Net-(JP1-Pad2)
- U9 pad 24: ~RD -> Net-(JP2-Pad2)
Routing:
- net GND: track 0.00 -> 803.6 mm, vias 0 -> 18
- net +5V: track 0.00 -> 656.3 mm, vias 0 -> 32
- net /A0: track 0.00 -> 363.8 mm, vias 0 -> 13
- net /D3: track 0.00 -> 337.0 mm, vias 0 -> 10
- net /D4: track 0.00 -> 321.2 mm, vias 0 -> 9
- net /D5: track 0.00 -> 320.4 mm, vias 0 -> 10
- net /D7: track 0.00 -> 303.5 mm, vias 0 -> 7
- net ~RD: track 0.00 -> 299.6 mm, vias 0 -> 7
- net /D6: track 0.00 -> 297.1 mm, vias 0 -> 7
- net ~RESET: track 0.00 -> 294.1 mm, vias 0 -> 10
- net /D1: track 0.00 -> 292.0 mm, vias 0 -> 12
- net /D2: track 0.00 -> 283.4 mm, vias 0 -> 10
- net /D0: track 0.00 -> 271.9 mm, vias 0 -> 11
- net /A1: track 0.00 -> 270.1 mm, vias 0 -> 10
- net /A13: track 0.00 -> 257.5 mm, vias 0 -> 10
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Other:
- board text added: "SINOPE V2.0 Hans Hübner (@hanshuebner) github.com/hanshuebner/sinope"
- board text removed: "IO GAL"
- board text removed: "MEMORY GAL"
- board text removed: "Oscillator"
- board text removed: "PWR Controller"
- board text removed: "RAM"
- board text removed: "RAM ADDR MUX"
- board text removed: "RESET"
- board text removed: "ROM"
- board text removed: "RS232 Level Converter"
- board text removed: "SINOPE V1.0 Hans Hübner (@hanshuebner) github.com/hanshuebner/sinope"
- board text removed: "Z80A CPU"
- board text removed: "Z80A CTC"
- board text removed: "Z80A PIO"
- board text removed: "Z80A SIO"

Commit message: Layout improved
Parts:
- moved C15 12.9 mm to (80.7, 47.2), turned to 180 degrees
- moved C21 7.34 mm to (166.0, 54.2), turned to 90 degrees
- moved C16 5.89 mm to (170.9, 83.6), turned to 270 degrees
- moved C22 1.87 mm to (93.8, 46.3), turned to 270 degrees
- moved C5 1.38 mm to (136.9, 95.2)
- moved C18 1.08 mm to (163.9, 38.9), turned to 270 degrees
- turned C19 to 180 degrees
Routing:
- net GND: track 803.6 -> 895.6 mm, vias 18 -> 35
- net CLK: track 224.1 -> 209.0 mm, vias 6 -> 5
- net ~M1: track 252.0 -> 264.8 mm, vias 7 -> 8
- net Net-(U4-Pad12): track 91.7 -> 100.7 mm, vias 2 -> 4
- net /A4: track 215.4 -> 206.7 mm, vias 6 -> 8
- net Net-(U4-Pad18): track 106.0 -> 114.6 mm, vias 2 -> 4
- net Net-(U4-Pad15): track 98.3 -> 106.3 mm, vias 2 -> 4
- net +5V: track 656.3 -> 664.1 mm, vias 32 -> 30
- net /A7: track 201.6 -> 194.3 mm, vias 12 -> 8
- net Net-(U4-Pad16): track 103.5 -> 110.0 mm, vias 2 -> 4
- net ~RESET: track 294.1 -> 300.4 mm, vias 10 -> 11
- net Net-(U4-Pad17): track 105.6 -> 111.5 mm, vias 2 -> 4
- net Net-(U4-Pad19): track 108.5 -> 104.8 mm, vias 2 -> 4
- net Net-(Q1-Pad2): track 5.35 -> 8.91 mm, vias 1 -> 0
- net Net-(J2-Pad7): track 30.1 -> 33.6 mm
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